File: hardware/mix/mix.sch (KiCad schematic (older format))
At the start: 6 parts, among them J1 LO, J2 IF, J3 RF, T1 ETC4-1-2TR, T2 ETC4-1-2TR

Commit message: Optimize Quad DDC, Gerber files
Parts:
- J1, J2, J3: symbol Connector:Conn_Coaxial -> CON-SMA-EDGE-S:CON-SMA-EDGE-S
Connections:
- net GND: now also J1.G1, J1.G2, J1.G3, J1.G4, J2.G1, J2.G2, J2.G3, J2.G4, J3.G1, J3.G2, J3.G3, J3.G4; no longer J1.2 (Ext), J2.2 (Ext), J3.2 (Ext)
Changed lines of the file:
@@
 Sheet 1 1
 Title "RF Mix"
-Date "2021-02-03"
+Date "2021-02-06"
 Rev ""
 Comp "R1CBU"
@@
 	7450 3650 7350 3650
 $Comp
-L Connector:Conn_Coaxial J1
+L CON-SMA-EDGE-S:CON-SMA-EDGE-S J1
 U 1 1 601B91E5
-P 3650 3250
-F 0 "J1" H 3578 3488 50  0000 C CNN
-F 1 "LO" H 3578 3397 50  0000 C CNN
-F 2 "Connector_Coaxial:SMA_Amphenol_132289_EdgeMount" H 3650 3250 50  0001 C CNN
-F 3 " ~" H 3650 3250 50  0001 C CNN
-	1    3650 3250
+P 3750 3350
+F 0 "J1" H 3500 3350 50  0000 C CNN
+F 1 "LO" H 3500 3450 50  0000 C CNN
+F 2 "Connector_Coaxial:SMA_Amphenol_132289_EdgeMount" H 3750 3350 50  0001 C CNN
+F 3 " ~" H 3750 3350 50  0001 C CNN
+	1    3750 3350
+	1    0    0    -1
+$EndComp
+$Comp
+L CON-SMA-EDGE-S:CON-SMA-EDGE-S J3
+U 1 1 601BB082
+P 7800 3350
+F 0 "J3" H 7550 3350 50  0000 L CNN
+F 1 "RF" H 7550 3450 50  0000 L CNN
+F 2 "Connector_Coaxial:SMA_Amphenol_132289_EdgeMount" H 7800 3350 50  0001 C CNN
+F 3 " ~" H 7800 3350 50  0001 C CNN
+	1    7800 3350
 	-1   0    0    -1
 $EndComp
 $Comp
-L Connector:Conn_Coaxial J3
-U 1 1 601BB082
-P 7750 3250
-F 0 "J3" H 7850 3225 50  0000 L CNN
-F 1 "RF" H 7850 3134 50  0000 L CNN
-F 2 "Connector_Coaxial:SMA_Amphenol_132289_EdgeMount" H 7750 3250 50  0001 C CNN
-F 3 " ~" H 7750 3250 50  0001 C CNN
-	1    7750 3250
-	1    0    0    -1
-$EndComp
-$Comp
-L Connector:Conn_Coaxial J2
+L CON-SMA-EDGE-S:CON-SMA-EDGE-S J2
 U 1 1 601BBC0E
-P 6950 4200
-F 0 "J2" H 7050 4175 50  0000 L CNN
-F 1 "IF" H 7050 4084 50  0000 L CNN
-F 2 "Connector_Coaxial:SMA_Amphenol_132289_EdgeMount" H 6950 4200 50  0001 C CNN
-F 3 " ~" H 6950 4200 50  0001 C CNN
-	1    6950 4200
-	1    0    0    -1
+P 6850 4300
+F 0 "J2" H 6600 4300 50  0000 L CNN
+F 1 "IF" H 6600 4400 50  0000 L CNN
+F 2 "Connector_Coaxial:SMA_Amphenol_132289_EdgeMount" H 6850 4300 50  0001 C CNN
+F 3 " ~" H 6850 4300 50  0001 C CNN
+	1    6850 4300
+	-1   0    0    -1
 $EndComp
 Wire Wire Line
 	3850 3250 4100 3250
 Wire Wire Line
-	7350 3250 7550 3250
-Wire Wire Line
-	7750 3450 7750 3650
-Wire Wire Line
-	7750 3650 7450 3650
+	7350 3250 7700 3250
+Wire Wire Line
+	7700 3350 7700 3650
 Connection ~ 7450 3650
 Wire Wire Line
-	3650 3450 3650 3650
-Wire Wire Line
-	3650 3650 4000 3650
+	3850 3350 3850 3650
+Wire Wire Line
+	3850 3650 4000 3650
 Connection ~ 4000 3650
 Wire Wire Line
@@
 L power:GND #PWR04
 U 1 1 601BF3F8
-P 6950 4600
-F 0 "#PWR04" H 6950 4350 50  0001 C CNN
-F 1 "GND" H 6955 4427 50  0000 C CNN
-F 2 "" H 6950 4600 50  0001 C CNN
-F 3 "" H 6950 4600 50  0001 C CNN
-	1    6950 4600
-	1    0    0    -1
-$EndComp
-Wire Wire Line
-	6950 4400 6950 4600
+P 6750 4650
+F 0 "#PWR04" H 6750 4400 50  0001 C CNN
+F 1 "GND" H 6755 4477 50  0000 C CNN
+F 2 "" H 6750 4650 50  0001 C CNN
+F 3 "" H 6750 4650 50  0001 C CNN
+	1    6750 4650
+	1    0    0    -1
+$EndComp
+Wire Wire Line
+	6750 4300 6750 4650
 Wire Wire Line
 	4750 3250 5400 3250
@@
 	1    0    0    -1
 $EndComp
+Wire Wire Line
+	7700 3650 7450 3650
 $EndSCHEMATC
