File: hardware/qddc/qddc.sch (KiCad schematic (older format))
At the start: 38 parts, among them IC1 FST3253MTCX, IC2 OPA2350UA, J1 In_cos, J2 In_sin, J3 In_RF, J4 PWR, J5 Out_I, J6 Out_Q, J7 Conn_01x03_Male, T1 ETC4-1-2TR

Commit message: Optimize Quad DDC, Gerber files
Parts:
- removed J5: Out_I, Connector_Coaxial:SMA_Amphenol_132289_EdgeMount, symbol Connector:Conn_Coaxial
- removed J6: Out_Q, Connector_Coaxial:SMA_Amphenol_132289_EdgeMount, symbol Connector:Conn_Coaxial
- J1, J2, J3: footprint Connector_Coaxial:SMA_Amphenol_132289_EdgeMount -> kicad:RFSOLUTIONS_CON-SMA-EDGE-S; symbol Connector:Conn_Coaxial -> CON-SMA-EDGE-S:CON-SMA-EDGE-S
Connections:
- net GND: now also J1.G1, J1.G2, J1.G3, J1.G4, J2.G1, J2.G2, J2.G3, J2.G4; no longer J1.2 (Ext), J2.2 (Ext)
- net at T1.4: now also J3.G1, J3.G2, J3.G3, J3.G4; no longer J3.1 (In)
- net at T1.5: now also J3.1; no longer J3.2 (Ext)
Other:
- moved on the sheet: C12, R12
Changed lines of the file:
@@
 Sheet 1 1
 Title "Quad DDC"
-Date "2021-02-04"
+Date "2021-02-06"
 Rev ""
 Comp "R1CBU"
@@
 $EndComp
 $Comp
-L Connector:Conn_Coaxial J3
+L CON-SMA-EDGE-S:CON-SMA-EDGE-S J3
 U 1 1 6015CF98
-P 1850 3650
-F 0 "J3" H 1950 3532 50  0000 L CNN
-F 1 "In_RF" H 1950 3623 50  0000 L CNN
-F 2 "Connector_Coaxial:SMA_Amphenol_132289_EdgeMount" H 1850 3650 50  0001 C CNN
-F 3 " ~" H 1850 3650 50  0001 C CNN
-	1    1850 3650
-	-1   0    0    1
+P 1950 3350
+F 0 "J3" H 1650 3350 50  0000 L CNN
+F 1 "In_RF" H 1550 3450 50  0000 L CNN
+F 2 "kicad:RFSOLUTIONS_CON-SMA-EDGE-S" H 1950 3350 50  0001 C CNN
+F 3 " ~" H 1950 3350 50  0001 C CNN
+	1    1950 3350
+	1    0    0    -1
 $EndComp
 Wire Wire Line
@@
 $EndComp
 $Comp
-L Connector:Conn_Coaxial J2
+L CON-SMA-EDGE-S:CON-SMA-EDGE-S J2
 U 1 1 6015DEEC
-P 1850 2750
-F 0 "J2" H 1949 2632 50  0000 L CNN
-F 1 "In_sin" H 1949 2723 50  0000 L CNN
-F 2 "Connector_Coaxial:SMA_Amphenol_132289_EdgeMount" H 1850 2750 50  0001 C CNN
-F 3 " ~" H 1850 2750 50  0001 C CNN
-	1    1850 2750
-	-1   0    0    -1
+P 1950 2850
+F 0 "J2" H 1650 2850 50  0000 L CNN
+F 1 "In_sin" H 1550 2950 50  0000 L CNN
+F 2 "kicad:RFSOLUTIONS_CON-SMA-EDGE-S" H 1950 2850 50  0001 C CNN
+F 3 " ~" H 1950 2850 50  0001 C CNN
+	1    1950 2850
+	1    0    0    -1
 $EndComp
 $Comp
@@
 L Device:R R12
 U 1 1 601C4F4D
-P 7350 1850
-F 0 "R12" V 7143 1850 50  0000 C CNN
-F 1 "100" V 7234 1850 50  0000 C CNN
-F 2 "Resistor_SMD:R_0805_2012Metric" V 7280 1850 50  0001 C CNN
-F 3 "~" H 7350 1850 50  0001 C CNN
-	1    7350 1850
-	-1   0    0    1
-$EndComp
-Wire Wire Line
-	7350 2150 7150 2150
+P 7650 2150
+F 0 "R12" V 7443 2150 50  0000 C CNN
+F 1 "100" V 7534 2150 50  0000 C CNN
+F 2 "Resistor_SMD:R_0805_2012Metric" V 7580 2150 50  0001 C CNN
+F 3 "~" H 7650 2150 50  0001 C CNN
+	1    7650 2150
+	0    -1   -1   0
+$EndComp
 $Comp
 L Device:R R13
@@
 F 3 "~" H 8800 2950 50  0001 C CNN
 	1    8800 2950
-	1    0    0    -1
-$EndComp
-$Comp
-L Connector:Conn_Coaxial J6
-U 1 1 601DF458
-P 9500 2700
-F 0 "J6" H 9600 2675 50  0000 L CNN
-F 1 "Out_Q" H 9600 2584 50  0000 L CNN
-F 2 "Connector_Coaxial:SMA_Amphenol_132289_EdgeMount" H 9500 2700 50  0001 C CNN
-F 3 " ~" H 9500 2700 50  0001 C CNN
-	1    9500 2700
-	1    0    0    -1
-$EndComp
-$Comp
-L Connector:Conn_Coaxial J5
-U 1 1 601E0053
-P 9500 1600
-F 0 "J5" H 9600 1575 50  0000 L CNN
-F 1 "Out_I" H 9600 1484 50  0000 L CNN
-F 2 "Connector_Coaxial:SMA_Amphenol_132289_EdgeMount" H 9500 1600 50  0001 C CNN
-F 3 " ~" H 9500 1600 50  0001 C CNN
-	1    9500 1600
-	1    0    0    -1
-$EndComp
-$Comp
-L power:GND #PWR0105
-U 1 1 601E9B5C
-P 9500 1800
-F 0 "#PWR0105" H 9500 1550 50  0001 C CNN
-F 1 "GND" H 9505 1627 50  0000 C CNN
-F 2 "" H 9500 1800 50  0001 C CNN
-F 3 "" H 9500 1800 50  0001 C CNN
-	1    9500 1800
-	1    0    0    -1
-$EndComp
-$Comp
-L power:GND #PWR0106
-U 1 1 601E9FDE
-P 9500 2900
-F 0 "#PWR0106" H 9500 2650 50  0001 C CNN
-F 1 "GND" H 9505 2727 50  0000 C CNN
-F 2 "" H 9500 2900 50  0001 C CNN
-F 3 "" H 9500 2900 50  0001 C CNN
-	1    9500 2900
 	1    0    0    -1
 $EndComp
@@
 	3150 2150 2050 2150
 $Comp
-L Connector:Conn_Coaxial J1
+L CON-SMA-EDGE-S:CON-SMA-EDGE-S J1
 U 1 1 6015E555
-P 1850 2150
-F 0 "J1" H 1950 2032 50  0000 L CNN
-F 1 "In_cos" H 1950 2123 50  0000 L CNN
-F 2 "Connector_Coaxial:SMA_Amphenol_132289_EdgeMount" H 1850 2150 50  0001 C CNN
-F 3 " ~" H 1850 2150 50  0001 C CNN
-	1    1850 2150
-	-1   0    0    -1
+P 1950 2250
+F 0 "J1" H 1650 2250 50  0000 L CNN
+F 1 "In_cos" H 1550 2350 50  0000 L CNN
+F 2 "kicad:RFSOLUTIONS_CON-SMA-EDGE-S" H 1950 2250 50  0001 C CNN
+F 3 " ~" H 1950 2250 50  0001 C CNN
+	1    1950 2250
+	1    0    0    -1
 $EndComp
 $Comp
 L power:GND #PWR0117
 U 1 1 60359400
-P 1850 2950
-F 0 "#PWR0117" H 1850 2700 50  0001 C CNN
-F 1 "GND" H 1855 2777 50  0000 C CNN
-F 2 "" H 1850 2950 50  0001 C CNN
-F 3 "" H 1850 2950 50  0001 C CNN
-	1    1850 2950
+P 2050 2950
+F 0 "#PWR0117" H 2050 2700 50  0001 C CNN
+F 1 "GND" H 2150 2950 50  0000 C CNN
+F 2 "" H 2050 2950 50  0001 C CNN
+F 3 "" H 2050 2950 50  0001 C CNN
+	1    2050 2950
 	1    0    0    -1
 $EndComp
@@
 L power:GND #PWR0118
 U 1 1 6035996A
-P 1850 2350
-F 0 "#PWR0118" H 1850 2100 50  0001 C CNN
-F 1 "GND" H 1855 2177 50  0000 C CNN
-F 2 "" H 1850 2350 50  0001 C CNN
-F 3 "" H 1850 2350 50  0001 C CNN
-	1    1850 2350
-	1    0    0    -1
-$EndComp
-Wire Wire Line
-	1850 3450 1850 3250
-Wire Wire Line
-	1850 3250 2300 3250
+P 2050 2350
+F 0 "#PWR0118" H 2050 2100 50  0001 C CNN
+F 1 "GND" H 2150 2350 50  0000 C CNN
+F 2 "" H 2050 2350 50  0001 C CNN
+F 3 "" H 2050 2350 50  0001 C CNN
+	1    2050 2350
+	1    0    0    -1
+$EndComp
+Wire Wire Line
+	2050 3250 2300 3250
 Wire Wire Line
 	8550 3350 8550 3950
@@
 Wire Wire Line
 	6900 3250 7150 3250
-Connection ~ 7150 2150
 $Comp
 L power:VAA #PWR0116
@@
 L Device:C C12
 U 1 1 6018E3D3
-P 9100 1600
-F 0 "C12" V 8848 1600 50  0000 C CNN
-F 1 "470nF" V 8939 1600 50  0000 C CNN
-F 2 "Capacitor_SMD:C_0805_2012Metric" H 9138 1450 50  0001 C CNN
-F 3 "~" H 9100 1600 50  0001 C CNN
-	1    9100 1600
+P 8550 2150
+F 0 "C12" V 8298 2150 50  0000 C CNN
+F 1 "470nF" V 8389 2150 50  0000 C CNN
+F 2 "Capacitor_SMD:C_0805_2012Metric" H 8588 2000 50  0001 C CNN
+F 3 "~" H 8550 2150 50  0001 C CNN
+	1    8550 2150
 	0    1    1    0
 $EndComp
@@
 	0    1    1    0
 $EndComp
-Wire Wire Line
-	9250 1600 9300 1600
 Wire Wire Line
 	8800 2700 8900 2700
@@
 $EndComp
 Wire Wire Line
-	9300 1600 9300 2150
-Wire Wire Line
-	9300 2150 9350 2150
-Connection ~ 9300 1600
-Wire Wire Line
 	9350 2350 9300 2350
 Wire Wire Line
 	9300 2350 9300 2700
-Connection ~ 9300 2700
 $Comp
 L power:GND #PWR0112
@@
 Wire Wire Line
 	9100 2250 9350 2250
-Wire Wire Line
-	7350 2150 7350 2000
-Wire Wire Line
-	7350 1700 7350 1600
-Wire Wire Line
-	7350 1600 8950 1600
 $Comp
 L Connector:Conn_01x03_Male J7
@@
 	-1   0    0    1
 $EndComp
+Wire Wire Line
+	7150 2150 7500 2150
+Connection ~ 7150 2150
+Wire Wire Line
+	8400 2150 7800 2150
+Wire Wire Line
+	8700 2150 9350 2150
+Wire Wire Line
+	2050 2250 2050 2350
+Wire Wire Line
+	2050 2950 2050 2850
+Wire Wire Line
+	2050 3650 2050 3350
 $EndSCHEMATC
