File: hardware/swr/swr.kicad_pcb (KiCad board)
At the start: 2 copper layers, 30 x 37 mm, 14 parts, among them J1 RF Out, J2 RF In, J3 Conn_01x03_Male, T1 BN43-202

Commit message: Update SWR
Parts:
- added H1: MountingHole_Pad, MountingHole:MountingHole_3.5mm_Pad, F.Cu at (161.3, 72.4)
- added H2: MountingHole_Pad, MountingHole:MountingHole_3.5mm_Pad, F.Cu at (161.3, 98.4)
Routing:
- net GND: vias 26 -> 24
Other:
- net class Default removed
- board text added: "SWR R1CBU"
